File: 104_LHv3.3.sch (KiCad schematic (older format))
At the start: 13 parts

Commit message: Fixed backwards LEDs
Connections:
- net GND: now also L1.1 (K), L2.1 (K); no longer L1.2 (A), L2.2 (A)
- net R1: now also L1.2 (A); no longer L1.1 (K)
- net R2: now also L2.2 (A); no longer L2.1 (K)
Other:
- moved on the sheet: L1, L2
Changed lines of the file:
@@
 EESchema Schematic File Version 4
+LIBS:104_LHv3.3-cache
 EELAYER 29 0
 EELAYER END
@@
 F 3 "" H 1425 3175 50  0001 C CNN
 	1    1425 3175
-	-1   0    0    1
+	1    0    0    -1
 $EndComp
 $Comp
@@
 F 3 "" H 1425 3425 50  0001 C CNN
 	1    1425 3425
-	-1   0    0    1
+	1    0    0    -1
 $EndComp
 Text Label 4625 3475 2    50   ~ 0
@@
 Text Label 2675 6775 2    50   ~ 0
 GND
+Text Label 1275 3425 2    50   ~ 0
+GND
+Text Label 1275 3175 2    50   ~ 0
+GND
+Text Label 2125 3175 0    50   ~ 0
+LED_00
+Text Label 2125 3425 0    50   ~ 0
+LED_01
+Wire Wire Line
+	9450 3800 10000 3800
+Wire Wire Line
+	9450 3950 10000 3950
+Wire Wire Line
+	9450 4100 10000 4100
+Wire Wire Line
+	9450 4250 10000 4250
+Wire Wire Line
+	9450 4400 10000 4400
+Wire Wire Line
+	9450 4550 10000 4550
+Wire Wire Line
+	9450 4700 10000 4700
+Wire Wire Line
+	9450 4850 10000 4850
+Wire Wire Line
+	9450 5000 10000 5000
+Wire Wire Line
+	9450 5150 10000 5150
+Wire Wire Line
+	9450 5300 10000 5300
+Wire Wire Line
+	9450 5450 10000 5450
+Wire Wire Line
+	9450 5600 10000 5600
+Wire Wire Line
+	9450 5750 10000 5750
+Wire Wire Line
+	9450 5900 10000 5900
+Wire Wire Line
+	9450 6050 10000 6050
+Wire Wire Line
+	9450 6200 10000 6200
+Wire Wire Line
+	9450 6350 10000 6350
+Wire Wire Line
+	9450 6500 10000 6500
+Wire Wire Line
+	9450 6650 10000 6650
+Wire Bus Line
+	12250 2175 12250 4500
 Wire Wire Line
 	1275 2975 1275 3175
@@
 Wire Wire Line
 	1275 3175 1275 3425
-Wire Wire Line
-	9450 3800 10000 3800
-Wire Wire Line
-	9450 3950 10000 3950
-Wire Wire Line
-	9450 4100 10000 4100
-Wire Wire Line
-	9450 4250 10000 4250
-Wire Wire Line
-	9450 4400 10000 4400
-Wire Wire Line
-	9450 4550 10000 4550
-Wire Wire Line
-	9450 4700 10000 4700
-Wire Wire Line
-	9450 4850 10000 4850
-Wire Wire Line
-	9450 5000 10000 5000
-Wire Wire Line
-	9450 5150 10000 5150
-Wire Wire Line
-	9450 5300 10000 5300
-Wire Wire Line
-	9450 5450 10000 5450
-Wire Wire Line
-	9450 5600 10000 5600
-Wire Wire Line
-	9450 5750 10000 5750
-Wire Wire Line
-	9450 5900 10000 5900
-Wire Wire Line
-	9450 6050 10000 6050
-Wire Wire Line
-	9450 6200 10000 6200
-Wire Wire Line
-	9450 6350 10000 6350
-Wire Wire Line
-	9450 6500 10000 6500
-Wire Wire Line
-	9450 6650 10000 6650
 Wire Wire Line
 	11950 4400 12450 4400
@@
 Wire Bus Line
 	5575 2175 12250 2175
-Wire Bus Line
-	12250 2175 12250 4500
 Wire Bus Line
 	4075 4075 4075 5675
@@
 Wire Bus Line
 	9650 3750 9650 6900
-Text Label 1275 3425 2    50   ~ 0
-GND
-Text Label 1275 3175 2    50   ~ 0
-GND
-Text Label 2125 3175 0    50   ~ 0
-LED_00
-Text Label 2125 3425 0    50   ~ 0
-LED_01
 $EndSCHEMATC
